File: KiCad/WLED_ESP32_Controller.kicad_pcb (KiCad board)
At the start: 2 copper layers, 62.2 x 30.5 mm, 24 parts, among them J1 Conn_01x06_Female, J2 Conn_01x04_Female, J3 Conn_01x07_Female, SW1 Reset, SW2 Flash, U1 AMS1117-3.3, U2 ESP32-WROOM-32, U3 SN74AHCT125D

Commit message: - update URL
Other:
- board text added: "WLED Controller V3 by Stefan Riese github.com/Hasenpups/WLED_ESP32_Controller Connect to WiFi SSID: WLED-AP PASS: wled1234"
- board text removed: "WLED Controller V3 by Stefan Riese github.com/Hasenpups/WLED_Controller_Public Connect to WiFi SSID: WLED-AP PASS: wled1234"
Changed lines of the file:
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@@
     (effects (font (size 1 1) (thickness 0.15)) (justify mirror))
   )
-  (gr_text "WLED Controller V3\nby Stefan Riese\ngithub.com/Hasenpups/WLED_Controller_Public\n\nConnect to WiFi\nSSID: WLED-AP\nPASS: wled1234" (at 139.7 108.966) (layer "B.SilkS")
+  (gr_text "WLED Controller V3\nby Stefan Riese\ngithub.com/Hasenpups/WLED_ESP32_Controller\n\nConnect to WiFi\nSSID: WLED-AP\nPASS: wled1234" (at 139.7 108.966) (layer "B.SilkS")
     (effects (font (size 1.2 1.2) (thickness 0.3)) (justify left mirror))
   )
